File: DMH_Dual_VCF_Diode_Ladder_PCB/Bridge.kicad_sch (KiCad schematic)
At the start: 8 parts, among them SW4 SW_SPDT_321, SW6 SW_SPDT_321

Commit message: Generated BoM
Parts:
- SW4, SW6: footprint (none) -> SynthStuff:Toggle_Switch_THT
Changed lines of the file:
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@@
 			)
 		)
-		(property "Footprint" ""
+		(property "Footprint" "SynthStuff:Toggle_Switch_THT"
 			(at 63.5 137.16 0)
 			(effects
@@
 			)
 		)
-		(property "Footprint" ""
+		(property "Footprint" "SynthStuff:Toggle_Switch_THT"
 			(at 63.5 111.76 0)
 			(effects
