File: DMH_Dual_VCF_Diode_Ladder_PCB/DMH_Dual_VCF_Diode_Ladder_PCB.kicad_pcb (KiCad board)
At the start: 2 copper layers, 96 x 157.5 mm, 68 parts, among them J0 Conn_01x01, J100 IDC_02x08, J200 IDC_02x05, J50 Conn_01x06, J60 Conn_01x06, SW1 SW_SPDT, SW2 SW_SPDT, SW3 SW_SPDT, SW4 SW_SPDT_321_OnOff, U1 TL074, U2 TL074

Commit message: Placed panel hole references on Main PCB
Parts:
- added C18: 100nF, Capacitor_THT:C_Disc_D4.3mm_W1.9mm_P5.00mm, F.Cu at (313.7, 161.2)
- added C21: 1uF, Capacitor_THT:C_Disc_D4.3mm_W1.9mm_P5.00mm, F.Cu at (330.3, 68.7)
- added C22: 1nF, Capacitor_THT:C_Disc_D4.3mm_W1.9mm_P5.00mm, F.Cu at (330.3, 72.2)
- added C23: 1nF, Capacitor_THT:C_Disc_D4.3mm_W1.9mm_P5.00mm, F.Cu at (330.3, 75.6)
- added C24: 1nF, Capacitor_THT:C_Disc_D4.3mm_W1.9mm_P5.00mm, F.Cu at (330.3, 79.0)
- added C25: 1nF, Capacitor_THT:C_Disc_D4.3mm_W1.9mm_P5.00mm, F.Cu at (330.3, 82.5)
- added C26: 1nF, Capacitor_THT:C_Disc_D4.3mm_W1.9mm_P5.00mm, F.Cu at (330.3, 86.0)
- added C27: 1uF, Capacitor_THT:C_Disc_D4.3mm_W1.9mm_P5.00mm, F.Cu at (330.3, 89.4)
- added C28: 1uF, Capacitor_THT:C_Disc_D4.3mm_W1.9mm_P5.00mm, F.Cu at (257.7, 142.2)
- added C29: 1nF, Capacitor_THT:C_Disc_D4.3mm_W1.9mm_P5.00mm, F.Cu at (257.7, 145.6)
- added C3: 100nF, Capacitor_THT:C_Disc_D4.3mm_W1.9mm_P5.00mm, F.Cu at (305.6, 137.1)
- added C30: 1nF, Capacitor_THT:C_Disc_D4.3mm_W1.9mm_P5.00mm, F.Cu at (257.7, 149.1)
- added C31: 1nF, Capacitor_THT:C_Disc_D4.3mm_W1.9mm_P5.00mm, F.Cu at (257.7, 152.5)
- added C32: 1nF, Capacitor_THT:C_Disc_D4.3mm_W1.9mm_P5.00mm, F.Cu at (257.7, 155.9)
- added C33: 1nF, Capacitor_THT:C_Disc_D4.3mm_W1.9mm_P5.00mm, F.Cu at (257.7, 159.4)
- added C34: 1uF, Capacitor_THT:C_Disc_D4.3mm_W1.9mm_P5.00mm, F.Cu at (257.7, 162.8)
- added C6: 100nF, Capacitor_THT:C_Disc_D4.3mm_W1.9mm_P5.00mm, F.Cu at (305.6, 147.4)
- added D15: 1N4148, Diode_THT:D_DO-35_SOD27_P7.62mm_Horizontal, F.Cu at (221.0, 142.2)
- added D16: 1N4148, Diode_THT:D_DO-35_SOD27_P7.62mm_Horizontal, F.Cu at (221.0, 145.8)
- added D17: 1N4148, Diode_THT:D_DO-35_SOD27_P7.62mm_Horizontal, F.Cu at (221.0, 149.3)
- added D18: 1N4148, Diode_THT:D_DO-35_SOD27_P7.62mm_Horizontal, F.Cu at (221.0, 152.8)
- added D19: 1N4148, Diode_THT:D_DO-35_SOD27_P7.62mm_Horizontal, F.Cu at (221.0, 156.4)
- added D20: 1N4148, Diode_THT:D_DO-35_SOD27_P7.62mm_Horizontal, F.Cu at (221.0, 159.9)
- added D21: 1N4148, Diode_THT:D_DO-35_SOD27_P7.62mm_Horizontal, F.Cu at (221.0, 163.5)
- added D22: 1N4148, Diode_THT:D_DO-35_SOD27_P7.62mm_Horizontal, F.Cu at (221.0, 167.1)
- added D23: 1N4148, Diode_THT:D_DO-35_SOD27_P7.62mm_Horizontal, F.Cu at (221.0, 170.6)
- added D3: LED, LED_THT:LED_D3.0mm, F.Cu at (279.4, 65.4)
- added D4: LED, LED_THT:LED_D3.0mm, F.Cu at (279.4, 70.8)
- added D5: LED, LED_THT:LED_D3.0mm, F.Cu at (279.4, 76.3)
- added J210: IDC_02x05, SynthStuff:IDC-Header_2x05_P2.54mm_Vertical_BackBone, F.Cu at (355.1, 48.8)
- added J70: Conn_01x06, Connector_PinSocket_2.54mm:PinSocket_1x06_P2.54mm_Vertical, F.Cu at (364.1, 45.0)
- added J80: Conn_01x06, Connector_PinSocket_2.54mm:PinSocket_1x06_P2.54mm_Vertical, F.Cu at (368.8, 45.0)
- added Q1: BC548, Package_TO_SOT_THT:TO-92L_Inline_Wide, F.Cu at (326.2, 123.7)
- added Q2: BC548, Package_TO_SOT_THT:TO-92L_Inline_Wide, F.Cu at (326.2, 129.3)
- added Q3: BC548, Package_TO_SOT_THT:TO-92L_Inline_Wide, F.Cu at (357.9, 117.1)
- added Q4: BC548, Package_TO_SOT_THT:TO-92L_Inline_Wide, F.Cu at (357.9, 122.8)
- added R25: 47k, Resistor_THT:R_Axial_DIN0207_L6.3mm_D2.5mm_P7.62mm_Horizontal, F.Cu at (257.3, 89.0)
- added R26: 100k, Resistor_THT:R_Axial_DIN0207_L6.3mm_D2.5mm_P7.62mm_Horizontal, F.Cu at (293.6, 44.7)
- added R27: 2k, Resistor_THT:R_Axial_DIN0207_L6.3mm_D2.5mm_P7.62mm_Horizontal, F.Cu at (293.6, 48.8)
- added R28: 100k, Resistor_THT:R_Axial_DIN0207_L6.3mm_D2.5mm_P7.62mm_Horizontal, F.Cu at (293.6, 52.8)
- added R29: 33k, Resistor_THT:R_Axial_DIN0207_L6.3mm_D2.5mm_P7.62mm_Horizontal, F.Cu at (293.6, 56.9)
- added R30: 27k, Resistor_THT:R_Axial_DIN0207_L6.3mm_D2.5mm_P7.62mm_Horizontal, F.Cu at (293.6, 60.9)
- added R31: 33k, Resistor_THT:R_Axial_DIN0207_L6.3mm_D2.5mm_P7.62mm_Horizontal, F.Cu at (293.6, 65.0)
- added R32: 33k, Resistor_THT:R_Axial_DIN0207_L6.3mm_D2.5mm_P7.62mm_Horizontal, F.Cu at (304.4, 44.7)
- added R33: 33k, Resistor_THT:R_Axial_DIN0207_L6.3mm_D2.5mm_P7.62mm_Horizontal, F.Cu at (304.4, 48.8)
- added R34: 33k, Resistor_THT:R_Axial_DIN0207_L6.3mm_D2.5mm_P7.62mm_Horizontal, F.Cu at (304.4, 52.8)
- added R35: 33k, Resistor_THT:R_Axial_DIN0207_L6.3mm_D2.5mm_P7.62mm_Horizontal, F.Cu at (304.4, 56.9)
- added R36: 33k, Resistor_THT:R_Axial_DIN0207_L6.3mm_D2.5mm_P7.62mm_Horizontal, F.Cu at (304.4, 60.9)
- added R37: 2k, Resistor_THT:R_Axial_DIN0207_L6.3mm_D2.5mm_P7.62mm_Horizontal, F.Cu at (304.4, 65.0)
- added R38: 100k, Resistor_THT:R_Axial_DIN0207_L6.3mm_D2.5mm_P7.62mm_Horizontal, F.Cu at (315.1, 44.7)
- added R39: 1k, Resistor_THT:R_Axial_DIN0207_L6.3mm_D2.5mm_P7.62mm_Horizontal, F.Cu at (315.1, 48.8)
- added R40: 1k, Resistor_THT:R_Axial_DIN0207_L6.3mm_D2.5mm_P7.62mm_Horizontal, F.Cu at (315.1, 52.8)
- added R41: 47K, Resistor_THT:R_Axial_DIN0207_L6.3mm_D2.5mm_P7.62mm_Horizontal, F.Cu at (315.1, 56.9)
- added R42: 100k, Resistor_THT:R_Axial_DIN0207_L6.3mm_D2.5mm_P7.62mm_Horizontal, F.Cu at (315.1, 60.9)
- added R43: 1k, Resistor_THT:R_Axial_DIN0207_L6.3mm_D2.5mm_P7.62mm_Horizontal, F.Cu at (315.1, 65.0)
- added R44: 100k, Resistor_THT:R_Axial_DIN0207_L6.3mm_D2.5mm_P7.62mm_Horizontal, F.Cu at (221.0, 118.2)
- added R45: 2k, Resistor_THT:R_Axial_DIN0207_L6.3mm_D2.5mm_P7.62mm_Horizontal, F.Cu at (221.0, 122.2)
- added R46: 100k, Resistor_THT:R_Axial_DIN0207_L6.3mm_D2.5mm_P7.62mm_Horizontal, F.Cu at (221.0, 126.2)
- added R47: 33k, Resistor_THT:R_Axial_DIN0207_L6.3mm_D2.5mm_P7.62mm_Horizontal, F.Cu at (221.0, 130.3)
- added R48: 27k, Resistor_THT:R_Axial_DIN0207_L6.3mm_D2.5mm_P7.62mm_Horizontal, F.Cu at (221.0, 134.3)
- added R49: 33k, Resistor_THT:R_Axial_DIN0207_L6.3mm_D2.5mm_P7.62mm_Horizontal, F.Cu at (221.0, 138.4)
- added R50: 33k, Resistor_THT:R_Axial_DIN0207_L6.3mm_D2.5mm_P7.62mm_Horizontal, F.Cu at (231.8, 118.2)
- added R51: 33k, Resistor_THT:R_Axial_DIN0207_L6.3mm_D2.5mm_P7.62mm_Horizontal, F.Cu at (231.8, 122.2)
- added R52: 33k, Resistor_THT:R_Axial_DIN0207_L6.3mm_D2.5mm_P7.62mm_Horizontal, F.Cu at (231.8, 126.2)
- added R53: 33k, Resistor_THT:R_Axial_DIN0207_L6.3mm_D2.5mm_P7.62mm_Horizontal, F.Cu at (231.8, 130.3)
- added R54: 33k, Resistor_THT:R_Axial_DIN0207_L6.3mm_D2.5mm_P7.62mm_Horizontal, F.Cu at (231.8, 134.3)
- added R55: 2k, Resistor_THT:R_Axial_DIN0207_L6.3mm_D2.5mm_P7.62mm_Horizontal, F.Cu at (231.8, 138.4)
- added R56: 100k, Resistor_THT:R_Axial_DIN0207_L6.3mm_D2.5mm_P7.62mm_Horizontal, F.Cu at (242.5, 118.2)
- added R57: 1k, Resistor_THT:R_Axial_DIN0207_L6.3mm_D2.5mm_P7.62mm_Horizontal, F.Cu at (242.5, 122.2)
- added R58: 1k, Resistor_THT:R_Axial_DIN0207_L6.3mm_D2.5mm_P7.62mm_Horizontal, F.Cu at (242.5, 126.2)
- added R59: 47K, Resistor_THT:R_Axial_DIN0207_L6.3mm_D2.5mm_P7.62mm_Horizontal, F.Cu at (242.5, 130.3)
- added R60: 100k, Resistor_THT:R_Axial_DIN0207_L6.3mm_D2.5mm_P7.62mm_Horizontal, F.Cu at (242.5, 134.3)
- added R61: 1k, Resistor_THT:R_Axial_DIN0207_L6.3mm_D2.5mm_P7.62mm_Horizontal, F.Cu at (242.5, 138.4)
- added R62: 33k, Resistor_THT:R_Axial_DIN0207_L6.3mm_D2.5mm_P7.62mm_Horizontal, F.Cu at (293.6, 103.0)
- added R64: 100k, Resistor_THT:R_Axial_DIN0207_L6.3mm_D2.5mm_P7.62mm_Horizontal, F.Cu at (293.6, 107.0)
- added R65: 100k, Resistor_THT:R_Axial_DIN0207_L6.3mm_D2.5mm_P7.62mm_Horizontal, F.Cu at (293.6, 111.0)
- added R66: 82k, Resistor_THT:R_Axial_DIN0207_L6.3mm_D2.5mm_P7.62mm_Horizontal, F.Cu at (293.6, 115.1)
- added R67: 100k, Resistor_THT:R_Axial_DIN0207_L6.3mm_D2.5mm_P7.62mm_Horizontal, F.Cu at (293.6, 119.2)
- added R68: 100R, Resistor_THT:R_Axial_DIN0207_L6.3mm_D2.5mm_P7.62mm_Horizontal, F.Cu at (293.6, 123.2)
- added R69: 10k, Resistor_THT:R_Axial_DIN0207_L6.3mm_D2.5mm_P7.62mm_Horizontal, F.Cu at (293.6, 127.2)
- added R70: 100R, Resistor_THT:R_Axial_DIN0207_L6.3mm_D2.5mm_P7.62mm_Horizontal, F.Cu at (293.6, 131.3)
- added R71: 100k, Resistor_THT:R_Axial_DIN0207_L6.3mm_D2.5mm_P7.62mm_Horizontal, F.Cu at (304.4, 103.0)
- added R72: 20k, Resistor_THT:R_Axial_DIN0207_L6.3mm_D2.5mm_P7.62mm_Horizontal, F.Cu at (304.4, 107.0)
- added R73: 20k, Resistor_THT:R_Axial_DIN0207_L6.3mm_D2.5mm_P7.62mm_Horizontal, F.Cu at (304.4, 111.0)
- added R74: 10k, Resistor_THT:R_Axial_DIN0207_L6.3mm_D2.5mm_P7.62mm_Horizontal, F.Cu at (304.4, 115.1)
- added R75: 10k, Resistor_THT:R_Axial_DIN0207_L6.3mm_D2.5mm_P7.62mm_Horizontal, F.Cu at (304.4, 119.2)
- added R76: 100k, Resistor_THT:R_Axial_DIN0207_L6.3mm_D2.5mm_P7.62mm_Horizontal, F.Cu at (304.4, 123.2)
- added R77: 100k, Resistor_THT:R_Axial_DIN0207_L6.3mm_D2.5mm_P7.62mm_Horizontal, F.Cu at (304.4, 127.2)
- added R78: 1k, Resistor_THT:R_Axial_DIN0207_L6.3mm_D2.5mm_P7.62mm_Horizontal, F.Cu at (304.4, 131.3)
- added R79: 33k, Resistor_THT:R_Axial_DIN0207_L6.3mm_D2.5mm_P7.62mm_Horizontal, F.Cu at (336.4, 103.0)
- added R81: 100k, Resistor_THT:R_Axial_DIN0207_L6.3mm_D2.5mm_P7.62mm_Horizontal, F.Cu at (336.4, 107.0)
- added R82: 100k, Resistor_THT:R_Axial_DIN0207_L6.3mm_D2.5mm_P7.62mm_Horizontal, F.Cu at (336.4, 111.0)
- added R83: 82k, Resistor_THT:R_Axial_DIN0207_L6.3mm_D2.5mm_P7.62mm_Horizontal, F.Cu at (336.4, 115.1)
- added R84: 100k, Resistor_THT:R_Axial_DIN0207_L6.3mm_D2.5mm_P7.62mm_Horizontal, F.Cu at (336.4, 119.2)
- added R85: 100R, Resistor_THT:R_Axial_DIN0207_L6.3mm_D2.5mm_P7.62mm_Horizontal, F.Cu at (336.4, 123.2)
- added R86: 10k, Resistor_THT:R_Axial_DIN0207_L6.3mm_D2.5mm_P7.62mm_Horizontal, F.Cu at (336.4, 127.2)
- added R87: 100R, Resistor_THT:R_Axial_DIN0207_L6.3mm_D2.5mm_P7.62mm_Horizontal, F.Cu at (336.4, 131.3)
- added R88: 100k, Resistor_THT:R_Axial_DIN0207_L6.3mm_D2.5mm_P7.62mm_Horizontal, F.Cu at (347.2, 103.0)
- added R89: 20k, Resistor_THT:R_Axial_DIN0207_L6.3mm_D2.5mm_P7.62mm_Horizontal, F.Cu at (347.2, 107.0)
- added R90: 20k, Resistor_THT:R_Axial_DIN0207_L6.3mm_D2.5mm_P7.62mm_Horizontal, F.Cu at (347.2, 111.0)
- added R91: 10k, Resistor_THT:R_Axial_DIN0207_L6.3mm_D2.5mm_P7.62mm_Horizontal, F.Cu at (347.2, 115.1)
- added R92: 10k, Resistor_THT:R_Axial_DIN0207_L6.3mm_D2.5mm_P7.62mm_Horizontal, F.Cu at (347.2, 119.2)
- added R93: 100k, Resistor_THT:R_Axial_DIN0207_L6.3mm_D2.5mm_P7.62mm_Horizontal, F.Cu at (347.2, 123.2)
- added R94: 100k, Resistor_THT:R_Axial_DIN0207_L6.3mm_D2.5mm_P7.62mm_Horizontal, F.Cu at (347.2, 127.2)
- added R95: 1k, Resistor_THT:R_Axial_DIN0207_L6.3mm_D2.5mm_P7.62mm_Horizontal, F.Cu at (347.2, 131.3)
- added R96: 5M, Resistor_THT:R_Axial_DIN0207_L6.3mm_D2.5mm_P7.62mm_Horizontal, F.Cu at (293.6, 167.4)
- added RV10: 50k, Potentiometer_THT:Potentiometer_Bourns_3296W_Vertical, F.Cu at (274.7, 85.2)
- added RV11: 100k, SynthStuff:Potentiometer_TT_P110KH1, F.Cu at (277.3, 61.0)
- added RV12: 100k, SynthStuff:Potentiometer_Alpha_RD901F-40-00D_Single_Vertical, F.Cu at (304.5, 86.1)
- added RV13: 50k, Potentiometer_THT:Potentiometer_Bourns_3296W_Vertical, F.Cu at (325.7, 84.8)
- added RV14: 100k, SynthStuff:Potentiometer_Alpha_RD901F-40-00D_Single_Vertical, F.Cu at (231.9, 159.5)
- added RV15: 50k, Potentiometer_THT:Potentiometer_Bourns_3296W_Vertical, F.Cu at (253.1, 158.3)
- added RV17: 50k, Potentiometer_THT:Potentiometer_Bourns_3296W_Vertical, F.Cu at (321.7, 123.7)
- added RV19: 100k, Potentiometer_THT:Potentiometer_Bourns_3296W_Vertical, F.Cu at (321.7, 130.1)
- added RV21: 50k, Potentiometer_THT:Potentiometer_Bourns_3296W_Vertical, F.Cu at (364.5, 104.2)
- added RV23: 100k, Potentiometer_THT:Potentiometer_Bourns_3296W_Vertical, F.Cu at (364.5, 110.6)
- added RV8: 50k, Potentiometer_THT:Potentiometer_Bourns_3296W_Vertical, F.Cu at (274.7, 78.8)
- added RV9: 100k, SynthStuff:Potentiometer_TT_P110KH1, F.Cu at (260.1, 61.0)
- added SW10: SW_DPDT_OnOn, SynthStuff:Toggle_Switch_2_Poles_TE, F.Cu at (258.4, 106.6)
- added SW5: SW_SPDT, SynthStuff:Toggle_Switch_TE, F.Cu at (243.2, 147.8)
- added SW6: SW_SPDT, SynthStuff:Toggle_Switch_TE, F.Cu at (251.8, 147.8)
- added SW7: SW_SPDT_OnOffOn, SynthStuff:Toggle_Switch_TE, F.Cu at (238.6, 106.4)
- added SW8: SW_SPDT_321, SynthStuff:Toggle_Switch_TE, F.Cu at (354.4, 160.0)
- added SW9: SW_SPDT_OnOffOn, SynthStuff:Toggle_Switch_TE, F.Cu at (247.2, 106.4)
- added U3: TL074, Package_DIP:DIP-14_W7.62mm_Socket, F.Cu at (326.4, 44.8)
- added U4: TL074, Package_DIP:DIP-14_W7.62mm_Socket, F.Cu at (338.2, 44.8)
- added U5: TL074, Package_DIP:DIP-14_W7.62mm_Socket, F.Cu at (253.8, 118.2)
- added U6: TL074, Package_DIP:DIP-14_W7.62mm_Socket, F.Cu at (265.6, 118.2)
- added U7: TL074, Package_DIP:DIP-14_W7.62mm_Socket, F.Cu at (315.6, 103.0)
- C1, C16, C17, C2, C4, C5, C8, C9, D1, D10, D11, D12, D13, D14, D2, D6, D7, D8, D9, J100, J200, J50, J60, R21, R4, U1, U2: moved to F.Cu
- C10, C11, C12, C13, C14: value 1nF -> 100nF; moved to F.Cu
- C15, C7: value 1uF -> 100nF; moved to F.Cu
- R1: value 27k -> 100k; moved to F.Cu
- R10: value 33k -> 47k; moved to F.Cu
- R11, R16: value 33k -> 100k; moved to F.Cu
- R12: value 33k -> 27k; moved to F.Cu
- R13, R14, R15: value 33k -> 3k3; moved to F.Cu
- R17: value 2k -> 27k; moved to F.Cu
- R18: value 100k -> 33k; moved to F.Cu
- R19, R23: value 1k -> 68k; moved to F.Cu
- R2: value 100k -> 27k; moved to F.Cu
- R20: value 1k -> 14k; moved to F.Cu
- R22: value 100k -> 68k; moved to F.Cu
- R24: value 68k -> 47k; moved to F.Cu
- R3: value 68k -> 33k; moved to F.Cu
- R5: value 100k -> 14k; moved to F.Cu
- R6: value 2k -> 33k; moved to F.Cu
- R7: value 14k -> 68k; moved to F.Cu
- R8: value 27k -> 68k; moved to F.Cu
- R9: value 100k -> 47k; moved to F.Cu
- RV2, RV4: value 100k -> 50k; footprint SynthStuff:Potentiometer_Alpha_RD901F-40-00D_Single_Vertical -> Potentiometer_THT:Potentiometer_Bourns_3296W_Vertical
- RV3, RV5: footprint SynthStuff:Potentiometer_Alpha_RD901F-40-00D_Single_Vertical -> SynthStuff:Potentiometer_TT_P110KH1
- RV6: value 50k -> 100k; footprint Potentiometer_THT:Potentiometer_Bourns_3296W_Vertical -> SynthStuff:Potentiometer_Alpha_RD901F-40-00D_Single_Vertical; moved to F.Cu
- SW1, SW2, SW3: footprint SynthStuff:Toggle_Switch_THT -> SynthStuff:Toggle_Switch_TE
- SW4: value SW_SPDT_321_OnOff -> SW_SPDT; footprint SynthStuff:Toggle_Switch_THT -> SynthStuff:Toggle_Switch_TE
- moved J200 283.2 mm to (334.2, 141.4)
- moved SW3 279.1 mm to (324.4, 74.3), turned to 0 degrees
- moved J0 265.2 mm to (320.2, 165.2)
- moved C1 262.5 mm to (322.7, 138.6), turned to 0 degrees
- moved J60 259.0 mm to (323.6, 177.8), turned to 90 degrees
- moved D1 249.7 mm to (305.9, 165.1), turned to 0 degrees
- moved C4 237.9 mm to (305.6, 140.5)
- moved SW1 237.3 mm to (307.1, 74.3), turned to 0 degrees
- moved C8 236.2 mm to (305.6, 154.3), turned to 0 degrees
- moved D6 232.8 mm to (293.6, 68.8), turned to 0 degrees
- moved C9 232.2 mm to (305.6, 157.8), turned to 0 degrees
- moved C7 230.6 mm to (305.6, 150.8)
- moved D2 225.6 mm to (305.9, 169.3), turned to 0 degrees
- moved J50 225.5 mm to (343.2, 155.0), turned to 0 degrees
- moved C2 220.1 mm to (322.7, 145.2), turned to 0 degrees
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Connections:
- C10 pad 1: Net-(D7-K) -> GND
- C10 pad 2: Net-(D13-K) -> -12V
- C11 pad 1: Net-(SW1-B) -> +12V
- C11 pad 2: Net-(D8-K) -> GND
- C12 pad 1: Net-(SW2-B) -> GND
- C12 pad 2: Net-(D10-A) -> -12V
- C13 pad 1: Net-(SW1-B) -> +12V
- C13 pad 2: Net-(D10-K) -> GND
- C14 pad 1: Net-(D11-K) -> GND
- C14 pad 2: Net-(D13-K) -> -12V
- C15 pad 1: Net-(C15-Pad1) -> +12V
- C15 pad 2: Net-(U2D-+) -> GND
- C16 pad 1: +12V -> GND
- C16 pad 2: GND -> -12V
- C17 pad 1: GND -> +12V
- C17 pad 2: -12V -> GND
- C4 pad 1: +12V -> GND
- C4 pad 2: GND -> -12V
- C5 pad 1: GND -> +12V
- C5 pad 2: -12V -> GND
- C7 pad 1: Net-(C7-Pad1) -> +12V
- C7 pad 2: Net-(C7-Pad2) -> GND
- C8 pad 1: +12V -> GND
- C8 pad 2: GND -> -12V
- C9 pad 1: GND -> +12V
- C9 pad 2: -12V -> GND
- D6 pad 2: Net-(D6-A) -> /CV Processing/CV A
- J100 pad 7a: /Inputs and Outputs/Bus CV In -> Net-(J100-Pin_7a)
- J100 pad 7b: /Inputs and Outputs/Bus CV In -> Net-(J100-Pin_7a)
- J200 pad 3: GND -> Net-(J200-Pin_3)
- J200 pad 8: GND -> unconnected-(J200-Pin_8-Pad8)
- J50 pad 1: /Core Circuit/Input -> /Core Circuit A/Input
- J50 pad 2: /Core Circuit/CV1 Input -> /CV Processing/CV1 A Input
- J50 pad 3: /Core Circuit/(Bus) CV2 Input -> /CV Processing/CV2 A Input
- J50 pad 4: /Core Circuit/CV3 Input -> /Inputs and Outputs A/Res CV Jack
- J50 pad 5: /Core Circuit/Output -> /Core Circuit A/Output
- J60 pad 3: Net-(J60-Pin_3) -> Net-(J200-Pin_3)
- R1 pad 2: -12V -> Net-(U1C--)
- R10 pad 1: Net-(SW3-B) -> GND
- R10 pad 2: Net-(U1D--) -> Net-(SW7-A)
- R11 pad 1: Net-(D6-K) -> Net-(R11-Pad1)
- R11 pad 2: Net-(U1D-+) -> Net-(U1C--)
- R12 pad 1: GND -> Net-(R12-Pad1)
- R12 pad 2: Net-(U1D-+) -> -12V
- R13 pad 1: Net-(U1D--) -> Net-(R13-Pad1)
- R13 pad 2: Net-(D12-K) -> Net-(D3-A)
- R14 pad 1: Net-(SW3-B) -> Net-(R14-Pad1)
- R14 pad 2: Net-(U1B--) -> Net-(D4-A)
- R15 pad 1: Net-(D6-K) -> Net-(R14-Pad1)
- R15 pad 2: Net-(U1B--) -> Net-(D5-A)
- R16 pad 1: Net-(U1B--) -> Net-(R16-Pad1)
- R16 pad 2: Net-(D7-A) -> Net-(U1C--)
- R17 pad 2: Net-(D7-A) -> -12V
- R18 pad 1: Net-(D13-K) -> /CV Processing/CV1 B Input
- R18 pad 2: Net-(D13-A) -> Net-(U2A--)
- R19 pad 2: GND -> Net-(U1C--)
- R2 pad 2: Net-(U1C--) -> -12V
- R20 pad 1: Net-(U2B--) -> Net-(U1C--)
- R20 pad 2: Net-(U2C--) -> /CV Processing/CV B
- R21 pad 1: Net-(U2C--) -> /CV Processing/CV2 B Input
- R21 pad 2: Net-(C15-Pad1) -> Net-(U2B--)
- R22 pad 1: GND -> Net-(R22-Pad1)
- R22 pad 2: Net-(U2D-+) -> Net-(U1C--)
- R23 pad 1: Net-(U2D--) -> Net-(U1C--)
- R23 pad 2: /Core Circuit/Output -> Net-(SW9-B)
- R24 pad 1: Net-(R24-Pad1) -> Net-(SW9-A)
- R24 pad 2: Net-(U1C--) -> /CV Processing/Bus CV A Input
- R3 pad 1: Net-(R3-Pad1) -> /CV Processing/CV1 A Input
- R3 pad 2: Net-(U1C--) -> Net-(U1A--)
- R5 pad 1: Net-(C7-Pad2) -> Net-(U1C--)
- R5 pad 2: Net-(U1A-+) -> /CV Processing/CV A
- R6 pad 1: GND -> /CV Processing/CV2 A Input
- R6 pad 2: Net-(U1A-+) -> Net-(U1B--)
- R7 pad 1: Net-(U1C--) -> Net-(R7-Pad1)
- R7 pad 2: Net-(D6-A) -> Net-(U1C--)
- R8 pad 1: Net-(D6-K) -> Net-(U1C--)
- R8 pad 2: GND -> Net-(SW7-B)
- R9 pad 1: -12V -> Net-(SW7-A)
- R9 pad 2: Net-(D6-K) -> /CV Processing/Bus CV A Input
- RV1 pad 1: GND -> Net-(R2-Pad1)
- RV1 pad 2: Net-(C7-Pad1) -> Net-(R1-Pad1)
- RV1 pad 3: /Core Circuit/Input -> +12V
- RV2 pad 1: Net-(R1-Pad1) -> Net-(U1A--)
- RV2 pad 2: Net-(R2-Pad1) -> Net-(R4-Pad1)
- RV2 pad 3: +12V -> Net-(R4-Pad1)
- RV3 pad 2: Net-(R3-Pad1) -> Net-(U1A-+)
- RV3 pad 3: /Core Circuit/CV1 Input -> /CV Processing/CV1 A Input
- RV4 pad 1: GND -> Net-(U1B--)
- RV4 pad 2: Net-(R4-Pad1) -> Net-(R7-Pad1)
- RV4 pad 3: /Core Circuit/(Bus) CV2 Input -> Net-(R7-Pad1)
- RV5 pad 2: Net-(U2A-+) -> Net-(U1B-+)
- RV5 pad 3: Net-(U2B--) -> /CV Processing/CV2 A Input
- RV6 pad 1: Net-(D13-A) -> Net-(R12-Pad1)
- RV6 pad 2: Net-(R19-Pad1) -> Net-(R11-Pad1)
- RV6 pad 3: Net-(R19-Pad1) -> +12V
- RV7 pad 1: GND -> Net-(R17-Pad1)
- RV7 pad 2: Net-(R24-Pad1) -> Net-(R16-Pad1)
- RV7 pad 3: /Core Circuit/CV3 Input -> +12V
- SW4 pad 1: Net-(J60-Pin_3) -> GND
- SW4 pad 2: /Inputs and Outputs/Bus CV In -> Net-(SW4-B)
- SW4 pad 3: unconnected-(SW4-A-Pad3) -> Net-(SW4-C)
- U1 pad 1: Net-(SW1-C) -> Net-(R4-Pad1)
- U1 pad 13: Net-(U1D--) -> Net-(SW1-C)
- U1 pad 14: Net-(D12-K) -> Net-(SW1-C)
- U1 pad 2: Net-(SW1-C) -> Net-(U1A--)
- U1 pad 5: GND -> Net-(U1B-+)
- U1 pad 7: Net-(R17-Pad1) -> Net-(R7-Pad1)
- U1 pad 8: Net-(D6-A) -> /CV Processing/CV A
- U2 pad 1: Net-(D13-K) -> Net-(R19-Pad1)
- U2 pad 12: Net-(U2D-+) -> /Core Circuit A/Res Input
- U2 pad 13: Net-(U2D--) -> Net-(D13-K)
- U2 pad 14: Net-(U2D--) -> Net-(D13-A)
- U2 pad 2: Net-(D13-A) -> Net-(U2A--)
- U2 pad 5: Net-(D10-A) -> Net-(U2B-+)
- U2 pad 7: Net-(U2B--) -> Net-(R22-Pad1)
- U2 pad 8: Net-(C15-Pad1) -> /CV Processing/CV B
- U2 pad 9: Net-(U2C--) -> Net-(U1C--)
Routing:
- net -12V: track 195.8 -> 0.00 mm
- net Net-(U1C--): track 177.0 -> 0.00 mm
- net Net-(SW1-C): track 170.4 -> 0.00 mm
- net +12V: track 134.2 -> 0.00 mm
- net Net-(SW3-B): track 122.8 -> 0.00 mm
- net /Inputs and Outputs/Bus CV In: track 111.3 -> 0.00 mm
- net /Core Circuit/Output: track 108.9 -> 0.00 mm
- net /Core Circuit/Input: track 105.0 -> 0.00 mm
- net Net-(D12-K): track 104.7 -> 0.00 mm
- net Net-(D13-K): track 97.4 -> 0.00 mm
- net /Core Circuit/CV1 Input: track 78.1 -> 0.00 mm
- net Net-(SW1-B): track 69.4 -> 0.00 mm
- net Net-(D6-K): track 66.4 -> 0.00 mm
- net Net-(J60-Pin_3): track 65.0 -> 0.00 mm
- net Net-(D10-A): track 57.6 -> 0.00 mm
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- removed copper zone on B.Cu, net GND
- removed copper zone on F.Cu, net GND
Other:
- board size 96 x 157.5 mm -> 146 x 175 mm

Commit message: Placed location dependent components on PCB
Parts:
- added RV16: 100k, SynthStuff:Potentiometer_TT_P110KH1, F.Cu at (80.5, 177.0)
- added RV18: 100k, SynthStuff:Potentiometer_Alpha_RD901F-40-00D_Single_Vertical, F.Cu at (77.5, 118.5)
- added RV20: 100k, SynthStuff:Potentiometer_TT_P110KH1, F.Cu at (114.5, 177.0)
- added RV22: 100k, SynthStuff:Potentiometer_Alpha_RD901F-40-00D_Single_Vertical, F.Cu at (117.5, 118.5)
- D3: value LED -> LED_Blue
- D4, D5: value LED -> LED_Red
- moved J80 303.2 mm to (109.8, 202.7)
- moved J50 275.4 mm to (69.5, 185.2)
- moved J70 272.5 mm to (130.5, 185.2)
- moved RV12 262.8 mm to (42.5, 106.5), turned to 90 degrees
- moved SW8 256.2 mm to (100.0, 190.2)
- moved SW1 251.9 mm to (64.0, 140.0)
- moved SW2 246.7 mm to (78.0, 140.0)
- moved SW3 241.5 mm to (92.0, 140.0)
- moved J60 234.6 mm to (90.3, 202.7), turned to 0 degrees
- moved RV5 226.3 mm to (48.5, 177.0)
- moved D4 213.3 mm to (66.7, 88.0)
- moved RV3 205.1 mm to (38.5, 145.0)
- moved SW10 188.5 mm to (100.0, 208.8)
- moved D3 184.5 mm to (98.7, 103.0)
- moved SW7 180.1 mm to (79.2, 190.2)
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
Commit message: Placed ICs and prepared passives
Parts:
- removed J200, J210: IDC_02x05, SynthStuff:IDC-Header_2x05_P2.54mm_Vertical_BackBone
- C1, C10, C11, C12, C13, C14, C15, C16, C17, C18, C2, C21, C22, C23, C24, C25, C26, C27, C28, C29, C3, C30, C31, C32, C33, C34, C4, C5, C6, C7, C8, C9, D1, D10, D11, D12, D13, D14, D15, D16, D17, D18, D19, D2, D20, D21, D22, D23, D6, D7, D8, D9, J100, Q1, Q2, Q3, Q4, R1, R10, R11, R12, R13, R14, R15, R16, R17, R18, R19, R2, R20, R21, R22, R23, R24, R25, R26, R27, R28, R29, R3, R30, R31, R32, R33, R34, R35, R36, R37, R38, R39, R4, R40, R41, R42, R43, R44, R45, R46, R47, R48, R49, R5, R50, R51, R52, R53, R54, R55, R56, R57, R58, R59, R6, R60, R61, R62, R64, R65, R66, R67, R68, R69, R7, R70, R71, R72, R73, R74, R75, R76, R77, R78, R79, R8, R81, R82, R83, R84, R85, R86, R87, R88, R89, R9, R90, R91, R92, R93, R94, R95, R96, RV10, RV13, RV15, RV17, RV19, RV2, RV21, RV23, RV4, RV8, U1, U2, U3, U4, U5, U6, U7: moved to B.Cu
- moved J0 247.1 mm to (30.0, 138.0)
- moved U7 213.4 mm to (103.8, 161.0), turned to 180 degrees
- moved C1 209.5 mm to (78.0, 47.2)
- moved U1 209.4 mm to (75.0, 60.0), turned to 180 degrees
- moved C3 196.8 mm to (74.8, 43.8), turned to -90 degrees
- moved D1 194.8 mm to (83.8, 54.1), turned to 90 degrees
- moved D2 172.7 mm to (116.2, 43.9), turned to -90 degrees
- moved C2 170.0 mm to (122.0, 47.2), turned to 180 degrees
- moved U2 164.0 mm to (132.5, 60.0), turned to 180 degrees
- moved U5 162.4 mm to (65.0, 110.0), turned to 180 degrees
- moved J100 156.6 mm to (108.9, 48.8), turned to 90 degrees
- moved C4 148.8 mm to (125.2, 48.8), turned to 90 degrees
- moved U3 143.0 mm to (90.0, 85.0), turned to 180 degrees
- moved U4 128.2 mm to (117.5, 85.0), turned to 180 degrees
- moved R71 99.0 mm to (199.1, 103.5), turned to 180 degrees
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
Commit message: Re-annotated OpAmps as per PCB layout
Connections:
- C27 pad 2: Net-(U3B-+) -> Net-(U3D-+)
- C34 pad 2: Net-(U5B-+) -> Net-(U4A-+)
- R1 pad 2: Net-(U1C--) -> Net-(U5B--)
- R11 pad 2: Net-(U1C--) -> Net-(U5B--)
- R16 pad 2: Net-(U1C--) -> Net-(U5B--)
- R18 pad 2: Net-(U2A--) -> Net-(U7A--)
- R19 pad 2: Net-(U1C--) -> Net-(U5B--)
- R20 pad 1: Net-(U1C--) -> Net-(U5B--)
- R21 pad 2: Net-(U2B--) -> Net-(U7B--)
- R22 pad 2: Net-(U1C--) -> Net-(U5B--)
- R23 pad 1: Net-(U1C--) -> Net-(U5B--)
- R26 pad 2: Net-(U1D-+) -> Net-(U5D-+)
- R27 pad 2: Net-(U1D-+) -> Net-(U5D-+)
- R29 pad 2: Net-(U4B-+) -> Net-(U5A-+)
- R3 pad 2: Net-(U1A--) -> Net-(U7D--)
- R31 pad 2: Net-(U3A--) -> Net-(U5C--)
- R32 pad 2: Net-(U3A--) -> Net-(U5C--)
- R33 pad 2: Net-(U4B--) -> Net-(U5A--)
- R34 pad 2: Net-(U4B-+) -> Net-(U5A-+)
- R35 pad 1: Net-(U3A--) -> Net-(U5C--)
- R36 pad 1: Net-(U4B--) -> Net-(U5A--)
- R39 pad 2: Net-(U4A--) -> Net-(U3C--)
- R4 pad 2: Net-(U1C--) -> Net-(U5B--)
- R41 pad 1: Net-(U4A--) -> Net-(U3C--)
- R42 pad 2: Net-(U3B-+) -> Net-(U3D-+)
- R43 pad 1: Net-(U3B--) -> Net-(U3D--)
- R44 pad 2: Net-(U3D-+) -> Net-(U6A-+)
- R45 pad 2: Net-(U3D-+) -> Net-(U6A-+)
- R47 pad 2: Net-(U6B-+) -> Net-(U6D-+)
- R49 pad 2: Net-(U5A--) -> Net-(U6B--)
- R5 pad 1: Net-(U1C--) -> Net-(U5B--)
- R50 pad 2: Net-(U5A--) -> Net-(U6B--)
- R51 pad 2: Net-(U6B--) -> Net-(U6D--)
- R52 pad 2: Net-(U6B-+) -> Net-(U6D-+)
- R53 pad 1: Net-(U5A--) -> Net-(U6B--)
- R54 pad 1: Net-(U6B--) -> Net-(U6D--)
- R57 pad 2: Net-(U6A--) -> Net-(U4B--)
- R59 pad 1: Net-(U6A--) -> Net-(U4B--)
- R6 pad 2: Net-(U1B--) -> Net-(U7C--)
- R60 pad 2: Net-(U5B-+) -> Net-(U4A-+)
- R61 pad 1: Net-(U5B--) -> Net-(U4A--)
- R62 pad 2: Net-(U5C--) -> Net-(U1D--)
- R64 pad 2: Net-(U5D--) -> Net-(U1B--)
- R65 pad 2: Net-(U5D--) -> Net-(U1B--)
- R66 pad 1: Net-(U5D--) -> Net-(U1B--)
- R7 pad 2: Net-(U1C--) -> Net-(U5B--)
- R74 pad 1: Net-(U7A--) -> Net-(U1C--)
- R75 pad 1: Net-(U7A-+) -> Net-(U1C-+)
- R76 pad 1: Net-(U7A-+) -> Net-(U1C-+)
- R77 pad 2: Net-(U7A--) -> Net-(U1C--)
- R79 pad 2: Net-(U6C--) -> Net-(U2A--)
- R8 pad 1: Net-(U1C--) -> Net-(U5B--)
- R81 pad 2: Net-(U6D--) -> Net-(U2C--)
- R82 pad 2: Net-(U6D--) -> Net-(U2C--)
- R83 pad 1: Net-(U6D--) -> Net-(U2C--)
- R91 pad 1: Net-(U7B--) -> Net-(U2B--)
- R92 pad 1: Net-(U7B-+) -> Net-(U2B-+)
- R93 pad 1: Net-(U7B-+) -> Net-(U2B-+)
- R94 pad 2: Net-(U7B--) -> Net-(U2B--)
- RV10 pad 1: Net-(U2B--) -> Net-(U7B--)
- RV11 pad 2: Net-(U2B-+) -> Net-(U7B-+)
- RV16 pad 2: Net-(U5C-+) -> Net-(U1D-+)
- RV17 pad 1: Net-(U5C--) -> Net-(U1D--)
- RV2 pad 1: Net-(U1A--) -> Net-(U7D--)
- RV20 pad 2: Net-(U6C-+) -> Net-(U2A-+)
- RV21 pad 1: Net-(U6C--) -> Net-(U2A--)
- RV3 pad 2: Net-(U1A-+) -> Net-(U7D-+)
- RV4 pad 1: Net-(U1B--) -> Net-(U7C--)
- RV5 pad 2: Net-(U1B-+) -> Net-(U7C-+)
- RV8 pad 1: Net-(U2A--) -> Net-(U7A--)
- RV9 pad 2: Net-(U2A-+) -> Net-(U7A-+)
- U1 pad 1: Net-(R4-Pad1) -> /CV Processing/Bus CV A Input
- U1 pad 10: GND -> Net-(U1C-+)
- U1 pad 13: Net-(SW1-C) -> Net-(U1D--)
- U1 pad 14: Net-(SW1-C) -> Net-(R64-Pad1)
- U1 pad 2: Net-(U1A--) -> /CV Processing/Bus CV A Input
- U1 pad 3: Net-(U1A-+) -> Net-(J100-Pin_7a)
- U1 pad 5: Net-(U1B-+) -> GND
- U1 pad 7: Net-(R7-Pad1) -> Net-(R66-Pad2)
- U1 pad 8: /CV Processing/CV A -> Net-(R77-Pad1)
- U2 pad 1: Net-(R19-Pad1) -> Net-(R81-Pad1)
- U2 pad 12: /Core Circuit A/Res Input -> GND
- U2 pad 13: Net-(D13-K) -> Net-(U2D--)
- U2 pad 14: Net-(D13-A) -> Net-(U2D--)
- U2 pad 7: Net-(R22-Pad1) -> Net-(R94-Pad1)
- U2 pad 8: /CV Processing/CV B -> Net-(R83-Pad2)
- U2 pad 9: Net-(U1C--) -> Net-(U2C--)
- U3 pad 1: Net-(R37-Pad1) -> Net-(D13-A)
- U3 pad 10: Net-(D10-A) -> GND
- U3 pad 13: Net-(SW4-C) -> Net-(U3D--)
- U3 pad 14: Net-(SW4-C) -> Net-(U3D--)
- U3 pad 2: Net-(U3A--) -> Net-(D13-K)
- U3 pad 3: GND -> /Core Circuit A/Res Input
- U3 pad 5: Net-(U3B-+) -> Net-(D10-A)
- U3 pad 6: Net-(U3B--) -> /Core Circuit A/Raw Output
- U3 pad 7: Net-(U3B--) -> /Core Circuit A/Raw Output
- U3 pad 8: /Core Circuit A/Raw Output -> Net-(C27-Pad1)
- U3 pad 9: /Core Circuit A/Raw Output -> Net-(U3C--)
- U4 pad 1: Net-(C27-Pad1) -> Net-(U4A--)
- U4 pad 3: GND -> Net-(U4A-+)
- U4 pad 5: Net-(U4B-+) -> GND
- U4 pad 7: Net-(D12-K) -> Net-(C34-Pad1)
- U5 pad 1: Net-(R55-Pad1) -> Net-(D12-K)
- U5 pad 10: Net-(U5C-+) -> GND
- U5 pad 12: GND -> Net-(U5D-+)
- U5 pad 13: Net-(U5D--) -> Net-(SW1-C)
- U5 pad 14: Net-(R66-Pad2) -> Net-(SW1-C)
- U5 pad 3: GND -> Net-(U5A-+)
- U5 pad 5: Net-(U5B-+) -> GND
- U5 pad 7: Net-(U5B--) -> /CV Processing/CV A
- U5 pad 8: Net-(R64-Pad1) -> Net-(R37-Pad1)
- U6 pad 1: Net-(C34-Pad1) -> Net-(SW4-C)
- U6 pad 10: Net-(U6C-+) -> GND
- U6 pad 12: GND -> Net-(U6D-+)
- U6 pad 14: Net-(R83-Pad2) -> Net-(D21-K)
- U6 pad 2: Net-(U6A--) -> Net-(SW4-C)
- U6 pad 3: GND -> Net-(U6A-+)
- U6 pad 5: Net-(U6B-+) -> GND
- U6 pad 7: Net-(D21-K) -> Net-(R55-Pad1)
- U6 pad 8: Net-(R81-Pad1) -> /CV Processing/CV B
- U6 pad 9: Net-(U6C--) -> Net-(U5B--)
- U7 pad 1: Net-(R77-Pad1) -> Net-(R19-Pad1)
- U7 pad 10: Net-(J100-Pin_7a) -> Net-(U7C-+)
- U7 pad 12: GND -> Net-(U7D-+)
- U7 pad 14: Net-(U7D--) -> Net-(R4-Pad1)
- U7 pad 7: Net-(R94-Pad1) -> Net-(R22-Pad1)
- U7 pad 8: /CV Processing/Bus CV A Input -> Net-(R7-Pad1)
- U7 pad 9: /CV Processing/Bus CV A Input -> Net-(U7C--)

Commit message: Component placement in progress
Parts:
- moved RV4 310.3 mm to (35.0, 171.0), turned to 90 degrees
- moved RV2 306.6 mm to (30.0, 134.0), turned to -90 degrees
- moved D7 264.8 mm to (30.5, 117.8), turned to 90 degrees
- moved D8 260.4 mm to (34.8, 117.8), turned to 90 degrees
- moved D9 256.3 mm to (38.9, 117.8), turned to 90 degrees
- moved D10 252.2 mm to (43.0, 117.8), turned to 90 degrees
- moved C25 251.9 mm to (30.5, 120.2), turned to -90 degrees
- moved R27 249.2 mm to (32.2, 99.3), turned to 90 degrees
- moved D11 248.1 mm to (47.2, 117.8), turned to 90 degrees
- moved C22 246.5 mm to (34.8, 125.2), turned to 90 degrees
- moved C21 246.0 mm to (37.0, 101.8), turned to -90 degrees
- moved R26 244.5 mm to (36.8, 99.3), turned to 90 degrees
- moved D12 244.0 mm to (51.5, 117.8), turned to 90 degrees
- moved C23 242.5 mm to (39.0, 125.2), turned to 90 degrees
- moved C24 238.4 mm to (43.2, 125.5), turned to 90 degrees
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Routing:
- added copper zone on B.Cu, net GND
- added copper zone on F.Cu, net GND

Commit message: Update DMH_Dual_VCF_Diode_Ladder_PCB.kicad_pcb
Parts:
- moved R31 230.6 mm to (50.5, 128.1), turned to 90 degrees
- moved RV13 230.0 mm to (94.5, 97.0), turned to 90 degrees
- moved D6 223.8 mm to (71.8, 120.4), turned to -90 degrees
- moved R36 220.3 mm to (50.5, 109.4), turned to -90 degrees
- moved R32 217.4 mm to (53.8, 128.1), turned to 90 degrees
- moved R33 216.6 mm to (53.8, 117.1), turned to 90 degrees
- moved R28 213.6 mm to (67.9, 131.0), turned to 0 degrees
- moved R35 212.8 mm to (58.1, 136.5)
- moved R37 212.3 mm to (58.1, 133.2)
- moved C27 210.9 mm to (78.8, 93.5), turned to 90 degrees
- moved R29 209.1 mm to (72.0, 117.1), turned to 90 degrees
- moved R30 206.3 mm to (74.8, 128.1), turned to 90 degrees
- moved D13 205.6 mm to (93.8, 92.1), turned to 90 degrees
- moved D14 205.0 mm to (97.0, 84.4), turned to -90 degrees
- moved R34 201.5 mm to (68.8, 117.1), turned to 90 degrees
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
Commit message: Component placement done
Parts:
- added R63: 20k, Resistor_THT:R_Axial_DIN0207_L6.3mm_D2.5mm_P7.62mm_Horizontal, B.Cu at (64.3, 73.0)
- added R80: 20k, Resistor_THT:R_Axial_DIN0207_L6.3mm_D2.5mm_P7.62mm_Horizontal, B.Cu at (135.4, 73.0)
- J50, J60, J70, J80: moved to B.Cu
- moved RV19 284.6 mm to (39.5, 62.2), turned to 90 degrees
- moved RV17 269.7 mm to (58.2, 47.2)
- moved Q2 252.5 mm to (58.0, 84.3), turned to 90 degrees
- moved Q1 250.1 mm to (64.2, 84.3), turned to 90 degrees
- moved R70 206.2 mm to (45.4, 73.0), turned to 0 degrees
- moved RV21 193.5 mm to (142.1, 47.5), turned to 0 degrees
- moved R95 192.7 mm to (114.5, 76.6), turned to 90 degrees
- moved R77 191.4 mm to (56.7, 69.8), turned to 0 degrees
- moved R64 191.4 mm to (63.8, 52.4), turned to -90 degrees
- moved R87 189.5 mm to (154.1, 73.0)
- moved R93 189.3 mm to (135.4, 66.5), turned to 0 degrees
- moved R81 189.3 mm to (136.2, 52.7), turned to -90 degrees
- moved R94 188.8 mm to (143.1, 69.8)
- moved R69 188.3 mm to (64.3, 76.2)
- moved Q3 186.8 mm to (135.4, 79.2), turned to -90 degrees
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