File: DMH_Dual_VCF_Diode_Ladder_PCB/DMH_Dual_VCF_Diode_Ladder_PCB.kicad_pcb (KiCad board)
At the start: 2 copper layers, 146 x 175 mm, 201 parts, among them J0 Conn_01x01, J100 IDC_02x08, J50 Conn_01x06, J60 Conn_01x06, J70 Conn_01x06, J80 Conn_01x06, Q1 BC548, Q2 BC548, Q3 BC548, Q4 BC548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

Commit message: Corrections before routing in progress
Parts:
- moved R1 5.00 mm to (31.2, 156.0)
- moved R16 5.00 mm to (168.8, 156.0)
- moved R19 4.25 mm to (168.8, 151.5)
- moved R4 4.25 mm to (31.2, 151.5)
- moved R12 1.75 mm to (96.2, 61.5)
- moved C3 1.25 mm to (74.8, 45.0)
- moved C4 1.25 mm to (125.2, 50.0)
- moved D1 1.00 mm to (83.8, 55.1)
- moved D2 1.00 mm to (116.2, 44.9)
- moved R23 0.25 mm to (161.2, 165.0)
- moved R8 0.25 mm to (38.8, 165.0)
Changed lines of the file:
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@@
 		(tags "potentiometer vertical TT P110KH1 single center detent")
 		(property "Reference" "RV9"
-			(at 2.5 -18.65 0)
+			(at -2 -18.5 0)
 			(layer "F.SilkS")
 			(effects
@@
 		)
 		(property "Value" "LED_Blue"
-			(at 1.27 2.96 0)
+			(at 1.27 -4.75 0)
 			(layer "F.SilkS")
 			(effects
@@
 		(tags "potentiometer vertical TT P110KH1 single center detent")
 		(property "Reference" "RV3"
-			(at 2.5 -18.65 0)
+			(at 7 -18.5 0)
 			(layer "F.SilkS")
 			(effects
@@
 		)
 		(property "Function" "Cutoff Common"
-			(at -2 2.5 0)
+			(at 13.5 2.5 0)
 			(layer "F.SilkS")
 			(effects
@@
 		(tags "Resistor Axial_DIN0207 series Axial Horizontal pin pitch 7.62mm 0.25W = 1/4W length 6.3mm diameter 2.5mm")
 		(property "Reference" "R58"
-			(at 3.81 2.37 0)
+			(at 9.31 0.75 90)
 			(layer "B.SilkS")
 			(effects
@@
 	(footprint "Resistor_THT:R_Axial_DIN0207_L6.3mm_D2.5mm_P7.62mm_Horizontal"
 		(layer "B.Cu")
-		(at 96.19 63.25)
+		(at 96.19 61.5)
 		(descr "Resistor, Axial_DIN0207 series, Axial, Horizontal, pin pitch=7.62mm, 0.25W = 1/4W, length*diameter=6.3*2.5mm^2, http://cdn-reichelt.de/documents/datenblatt/B400/1_4W%23YAG.pdf")
 		(tags "Resistor Axial_DIN0207 series Axial Horizontal pin pitch 7.62mm 0.25W = 1/4W length 6.3mm diameter 2.5mm")
@@
 	(footprint "Resistor_THT:R_Axial_DIN0207_L6.3mm_D2.5mm_P7.62mm_Horizontal"
 		(layer "B.Cu")
-		(at 168.81 155.75 180)
+		(at 168.81 151.5 180)
 		(descr "Resistor, Axial_DIN0207 series, Axial, Horizontal, pin pitch=7.62mm, 0.25W = 1/4W, length*diameter=6.3*2.5mm^2, http://cdn-reichelt.de/documents/datenblatt/B400/1_4W%23YAG.pdf")
 		(tags "Resistor Axial_DIN0207 series Axial Horizontal pin pitch 7.62mm 0.25W = 1/4W length 6.3mm diameter 2.5mm")
@@
 	(footprint "Capacitor_THT:C_Disc_D4.3mm_W1.9mm_P5.00mm"
 		(layer "B.Cu")
-		(at 125.25 48.75 90)
+		(at 125.25 50 90)
 		(descr "C, Disc series, Radial, pin pitch=5.00mm, , diameter*width=4.3*1.9mm^2, Capacitor, http://www.vishay.com/docs/45233/krseries.pdf")
 		(tags "C Disc series Radial pin pitch 5.00mm  diameter 4.3mm width 1.9mm Capacitor")
@@
 	(footprint "Resistor_THT:R_Axial_DIN0207_L6.3mm_D2.5mm_P7.62mm_Horizontal"
 		(layer "B.Cu")
-		(at 31.19 151)
+		(at 31.19 156)
 		(descr "Resistor, Axial_DIN0207 series, Axial, Horizontal, pin pitch=7.62mm, 0.25W = 1/4W, length*diameter=6.3*2.5mm^2, http://cdn-reichelt.de/documents/datenblatt/B400/1_4W%23YAG.pdf")
 		(tags "Resistor Axial_DIN0207 series Axial Horizontal pin pitch 7.62mm 0.25W = 1/4W length 6.3mm diameter 2.5mm")
@@
 	(footprint "Capacitor_THT:C_Disc_D4.3mm_W1.9mm_P5.00mm"
 		(layer "B.Cu")
-		(at 74.75 43.75 -90)
+		(at 74.75 45 -90)
 		(descr "C, Disc series, Radial, pin pitch=5.00mm, , diameter*width=4.3*1.9mm^2, Capacitor, http://www.vishay.com/docs/45233/krseries.pdf")
 		(tags "C Disc series Radial pin pitch 5.00mm  diameter 4.3mm width 1.9mm Capacitor")
@@
 	(footprint "Diode_THT:D_DO-41_SOD81_P10.16mm_Horizontal"
 		(layer "B.Cu")
-		(at 83.75 54.08 90)
+		(at 83.75 55.08 90)
 		(descr "Diode, DO-41_SOD81 series, Axial, Horizontal, pin pitch=10.16mm, , length*diameter=5.2*2.7mm^2, , http://www.diodes.com/_files/packages/DO-41%20(Plastic).pdf")
 		(tags "Diode DO-41_SOD81 series Axial Horizontal pin pitch 10.16mm  length 5.2mm diameter 2.7mm")
@@
 	(footprint "Resistor_THT:R_Axial_DIN0207_L6.3mm_D2.5mm_P7.62mm_Horizontal"
 		(layer "B.Cu")
-		(at 161.19 165.25)
+		(at 161.19 165)
 		(descr "Resistor, Axial_DIN0207 series, Axial, Horizontal, pin pitch=7.62mm, 0.25W = 1/4W, length*diameter=6.3*2.5mm^2, http://cdn-reichelt.de/documents/datenblatt/B400/1_4W%23YAG.pdf")
 		(tags "Resistor Axial_DIN0207 series Axial Horizontal pin pitch 7.62mm 0.25W = 1/4W length 6.3mm diameter 2.5mm")
@@
 	(footprint "Resistor_THT:R_Axial_DIN0207_L6.3mm_D2.5mm_P7.62mm_Horizontal"
 		(layer "B.Cu")
-		(at 168.81 151 180)
+		(at 168.81 156 180)
 		(descr "Resistor, Axial_DIN0207 series, Axial, Horizontal, pin pitch=7.62mm, 0.25W = 1/4W, length*diameter=6.3*2.5mm^2, http://cdn-reichelt.de/documents/datenblatt/B400/1_4W%23YAG.pdf")
 		(tags "Resistor Axial_DIN0207 series Axial Horizontal pin pitch 7.62mm 0.25W = 1/4W length 6.3mm diameter 2.5mm")
@@
 	(footprint "Diode_THT:D_DO-41_SOD81_P10.16mm_Horizontal"
 		(layer "B.Cu")
-		(at 116.25 43.92 -90)
+		(at 116.25 44.92 -90)
 		(descr "Diode, DO-41_SOD81 series, Axial, Horizontal, pin pitch=10.16mm, , length*diameter=5.2*2.7mm^2, , http://www.diodes.com/_files/packages/DO-41%20(Plastic).pdf")
 		(tags "Diode DO-41_SOD81 series Axial Horizontal pin pitch 10.16mm  length 5.2mm diameter 2.7mm")
@@
 		(tags "Resistor Axial_DIN0207 series Axial Horizontal pin pitch 7.62mm 0.25W = 1/4W length 6.3mm diameter 2.5mm")
 		(property "Reference" "R40"
-			(at 9.31 -0.5 -90)
+			(at 9.31 -0.75 -90)
 			(layer "B.SilkS")
 			(effects
@@
 	(footprint "Resistor_THT:R_Axial_DIN0207_L6.3mm_D2.5mm_P7.62mm_Horizontal"
 		(layer "B.Cu")
-		(at 38.81 165.25 180)
+		(at 38.81 165 180)
 		(descr "Resistor, Axial_DIN0207 series, Axial, Horizontal, pin pitch=7.62mm, 0.25W = 1/4W, length*diameter=6.3*2.5mm^2, http://cdn-reichelt.de/documents/datenblatt/B400/1_4W%23YAG.pdf")
 		(tags "Resistor Axial_DIN0207 series Axial Horizontal pin pitch 7.62mm 0.25W = 1/4W length 6.3mm diameter 2.5mm")
@@
 	(footprint "Resistor_THT:R_Axial_DIN0207_L6.3mm_D2.5mm_P7.62mm_Horizontal"
 		(layer "B.Cu")
-		(at 31.19 155.75)
+		(at 31.19 151.5)
 		(descr "Resistor, Axial_DIN0207 series, Axial, Horizontal, pin pitch=7.62mm, 0.25W = 1/4W, length*diameter=6.3*2.5mm^2, http://cdn-reichelt.de/documents/datenblatt/B400/1_4W%23YAG.pdf")
 		(tags "Resistor Axial_DIN0207 series Axial Horizontal pin pitch 7.62mm 0.25W = 1/4W length 6.3mm diameter 2.5mm")

Commit message: Routing ongoing
Routing:
- net +12V: track 0.00 -> 487.1 mm
- net -12V: track 0.00 -> 486.1 mm
- net Net-(U2A-+): track 0.00 -> 128.7 mm
- net /Inputs and Outputs B/Res CV Jack: track 0.00 -> 128.3 mm
- net Net-(U5B--): track 0.00 -> 127.4 mm
- net Net-(D22-A): track 0.00 -> 112.3 mm
- net Net-(R16-Pad1): track 0.00 -> 109.6 mm
- net /Core Circuit B/Input: track 0.00 -> 90.4 mm
- net Net-(D18-K): track 0.00 -> 68.1 mm
- net Net-(D5-A): track 0.00 -> 57.5 mm
- net Net-(R80-Pad1): track 0.00 -> 52.8 mm
- net Net-(D16-A): track 0.00 -> 43.7 mm
- net Net-(R82-Pad1): track 0.00 -> 41.7 mm
- net Net-(U6A-+): track 0.00 -> 38.7 mm
- net Net-(R94-Pad1): track 0.00 -> 34.8 mm
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
Commit message: Routing in progress
Routing:
- net Net-(U5B--): track 127.4 -> 272.9 mm
- net /Inputs and Outputs A/Res CV Jack: track 0.00 -> 126.8 mm
- net Net-(D13-A): track 19.3 -> 135.5 mm
- net Net-(R13-Pad1): track 0.00 -> 99.4 mm
- net Net-(R14-Pad1): track 0.00 -> 99.1 mm
- net Net-(R1-Pad1): track 0.00 -> 94.9 mm
- net /Core Circuit A/Input: track 0.00 -> 87.8 mm
- net Net-(D10-A): track 11.3 -> 75.8 mm
- net +12V: track 487.1 -> 550.0 mm
- net Net-(U5D-+): track 0.00 -> 47.8 mm
- net /CV Processing/Bus CV A Input: track 2.54 -> 49.1 mm
- net Net-(D7-A): track 0.00 -> 43.5 mm
- net /Core Circuit A/Raw Output: track 0.00 -> 39.2 mm
- net Net-(SW1-B): track 0.00 -> 33.5 mm
- net Net-(U3D--): track 0.00 -> 28.1 mm
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
Commit message: Finished routing
Parts:
- moved R11 0.50 mm to (103.8, 81.0)
Connections:
- J60 pad 1: Net-(J60-Pin_1) -> unconnected-(J60-Pin_1-Pad1)
- J60 pad 2: Net-(J60-Pin_2) -> unconnected-(J60-Pin_2-Pad2)
- J60 pad 3: Net-(J60-Pin_3) -> unconnected-(J60-Pin_3-Pad3)
- J60 pad 4: Net-(J60-Pin_4) -> unconnected-(J60-Pin_4-Pad4)
- J60 pad 5: Net-(J60-Pin_5) -> unconnected-(J60-Pin_5-Pad5)
- J60 pad 6: GND -> unconnected-(J60-Pin_6-Pad6)
- SW1 pad 1: GND -> Net-(SW1-A)
- SW1 pad 3: Net-(SW1-C) -> GND
- SW2 pad 1: GND -> Net-(SW1-A)
- SW2 pad 3: Net-(SW1-C) -> GND
- SW3 pad 1: GND -> Net-(SW1-A)
- SW3 pad 3: Net-(SW1-C) -> GND
- SW4 pad 1: GND -> Net-(SW4-A)
- SW4 pad 3: Net-(SW4-C) -> GND
- SW5 pad 1: GND -> Net-(SW4-A)
- SW5 pad 3: Net-(SW4-C) -> GND
- SW6 pad 1: GND -> Net-(SW4-A)
- SW6 pad 3: Net-(SW4-C) -> GND
- U5 pad 13: Net-(SW1-C) -> Net-(SW1-A)
- U5 pad 14: Net-(SW1-C) -> Net-(SW1-A)
- U6 pad 1: Net-(SW4-C) -> Net-(SW4-A)
- U6 pad 2: Net-(SW4-C) -> Net-(SW4-A)
Routing:
- net /CV Processing/CV2 A Input: track 13.0 -> 147.5 mm
- net Net-(U1D-+): track 0.00 -> 129.6 mm
- net /CV Processing/Bus CV A Input: track 49.1 -> 177.2 mm
- net /Inputs and Outputs A/Res CV Jack: track 126.8 -> 247.6 mm
- net /CV Processing/CV1 A Input: track 0.00 -> 117.1 mm
- net /CV Processing/Link Switch: track 0.00 -> 115.9 mm
- net /Core Circuit A/Output: track 0.00 -> 113.9 mm
- net /Core Circuit B/Output: track 0.00 -> 113.8 mm
- net /CV Processing/CV B: track 4.80 -> 117.8 mm
- net /CV Processing/CV A: track 8.83 -> 106.2 mm
- net Net-(U5B--): track 272.9 -> 360.9 mm
- net Net-(SW4-A): track 0.00 -> 85.2 mm
- net Net-(U7A-+): track 0.00 -> 78.1 mm
- net Net-(R19-Pad1): track 20.9 -> 98.2 mm
- net Net-(U7D--): track 12.5 -> 87.9 mm
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