File: DMH_Dual_VCF_Diode_Ladder_PCB/Resonance_B_CV.kicad_sch (KiCad schematic)
At the start: 24 parts, among them Q1 BC548, Q2 BC548, U3 TL074

Commit message: Concluded core and resonance circuits design
Parts:
- RV12: renamed from RV9; Function Zero adj Res A -> Zero adj Res B
- RV13: renamed from RV11; Function Res A CV Amt -> Res B CV Amt
- RV15: renamed from RV8; Function Res A -> Res B
- renumbered Q1 to Q3, Q2 to Q4, R27 to R32, R28 to R45, R29 to R46, R30 to R47, R33 to R48, R34 to R49, R35 to R50, R36 to R51, R37 to R52, R38 to R53, R39 to R54, R40 to R55, R41 to R56, R42 to R57, R31 to R58, R43 to R59, R44 to R60, RV10 to RV14, U3 to U4

Commit message: Reannotated whole schematic
OpAmp annotation is still tentative.
Parts:
- renumbered R51 to R79, R58 to R80, R52 to R81, R60 to R82, R59 to R83, R53 to R84, R55 to R85, R57 to R86, R56 to R87, R54 to R88, R32 to R89, R45 to R90, R47 to R91, R49 to R92, R50 to R93, R46 to R94, R48 to R95, RV13 to RV20, RV12 to RV21, RV15 to RV22, RV14 to RV23, U4 to U6, U4 to U8
Connections:
- net GND: now also U6.12 (+); no longer U6.10 (+)
- net at RV20.2: now also U6.3 (+); no longer U6.5 (+)
- net at R79.2, RV21.1: now also U6.2 (-); no longer U6.6 (-)
- net at R81.1, RV21.2, RV21.3: now also U6.1; no longer U6.7
- net at R92.1, R93.1: now also U8.10 (+); no longer U8.12 (+)
- net at R83.2, R86.1: now also U6.14; no longer U6.8
- net at R91.1, R94.2: now also U8.9 (-); no longer U8.13 (-)
- net at R94.1, R95.2: now also U8.8; no longer U8.14
- net at R81.2, R82.2, R83.1: now also U6.13 (-); no longer U6.9 (-)

Commit message: Reannotated OpAmps and cleared errors
Parts:
- renumbered U8 to U7
Connections:
- net at R81.1, RV21.2, RV21.3: now also U6.8; no longer U6.1
- net at R79.2, RV21.1: now also U6.9 (-); no longer U6.2 (-)
- net at RV20.2: now also U6.10 (+); no longer U6.3 (+)
- net at R92.1, R93.1: now also U7.5 (+); no longer U7.10 (+)
- net at R94.1, R95.2: now also U7.7; no longer U7.8
- net at R91.1, R94.2: now also U7.6 (-); no longer U7.9 (-)
Changed lines of the file:
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@@
 		(at 95.25 88.9 0)
 		(mirror x)
-		(unit 1)
+		(unit 3)
 		(exclude_from_sim no)
 		(in_bom yes)
@@
 				(path "/58f4306d-5387-4983-bb08-41a2313fd315/f0045393-e1d0-4de8-baba-b9053cd8a11d"
 					(reference "U6")
-					(unit 1)
+					(unit 3)
 				)
 			)
@@
 		(at 234.95 50.8 0)
 		(mirror x)
-		(unit 3)
-		(exclude_from_sim no)
-		(in_bom yes)
-		(on_board yes)
-		(dnp no)
-		(property "Reference" "U8"
+		(unit 2)
+		(exclude_from_sim no)
+		(in_bom yes)
+		(on_board yes)
+		(dnp no)
+		(property "Reference" "U7"
 			(at 234.95 60.96 0)
 			(effects
@@
 			(project "DMH_Dual_VCF_Diode_Ladder_PCB"
 				(path "/58f4306d-5387-4983-bb08-41a2313fd315/f0045393-e1d0-4de8-baba-b9053cd8a11d"
-					(reference "U8")
-					(unit 3)
-				)
-			)
+					(reference "U7")
+					(unit 2)
+				)
+			)

Commit message: Re-annotated OpAmps as per PCB layout
Parts:
- renumbered U6 to U2, U7 to U2
Connections:
- net GND: now also U2.10 (+); no longer U2.12 (+)
- net at RV20.2: now also U2.3 (+); no longer U2.10 (+)
- net at R81.1, RV21.2, RV21.3: now also U2.1; no longer U2.8
- net at R79.2, RV21.1: now also U2.2 (-); no longer U2.9 (-)
- net at R83.2, R86.1: now also U2.8; no longer U2.14
- net at R81.2, R82.2, R83.1: now also U2.9 (-); no longer U2.13 (-)
Changed lines of the file:
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@@
 		(at 95.25 88.9 0)
 		(mirror x)
-		(unit 3)
-		(exclude_from_sim no)
-		(in_bom yes)
-		(on_board yes)
-		(dnp no)
-		(property "Reference" "U6"
+		(unit 1)
+		(exclude_from_sim no)
+		(in_bom yes)
+		(on_board yes)
+		(dnp no)
+		(property "Reference" "U2"
 			(at 95.25 99.06 0)
 			(effects
@@
 			(project "DMH_Dual_VCF_Diode_Ladder_PCB"
 				(path "/58f4306d-5387-4983-bb08-41a2313fd315/f0045393-e1d0-4de8-baba-b9053cd8a11d"
-					(reference "U6")
-					(unit 3)
+					(reference "U2")
+					(unit 1)
 				)
 			)
@@
 		(on_board yes)
 		(dnp no)
-		(property "Reference" "U7"
+		(property "Reference" "U2"
 			(at 234.95 60.96 0)
 			(effects
@@
 			(project "DMH_Dual_VCF_Diode_Ladder_PCB"
 				(path "/58f4306d-5387-4983-bb08-41a2313fd315/f0045393-e1d0-4de8-baba-b9053cd8a11d"
-					(reference "U7")
+					(reference "U2")
 					(unit 2)
 				)
@@
 		(at 138.43 127 0)
 		(mirror x)
-		(unit 4)
-		(exclude_from_sim no)
-		(in_bom yes)
-		(on_board yes)
-		(dnp no)
-		(property "Reference" "U6"
+		(unit 3)
+		(exclude_from_sim no)
+		(in_bom yes)
+		(on_board yes)
+		(dnp no)
+		(property "Reference" "U2"
 			(at 138.43 137.16 0)
 			(effects
@@
 			(project "DMH_Dual_VCF_Diode_Ladder_PCB"
 				(path "/58f4306d-5387-4983-bb08-41a2313fd315/f0045393-e1d0-4de8-baba-b9053cd8a11d"
-					(reference "U6")
-					(unit 4)
-				)
-			)
+					(reference "U2")
+					(unit 3)
+				)
+			)
