File: DMH_Dual_VCF_Diode_Ladder_PANEL/DMH_Dual_VCF_Diode_Ladder_PANEL.kicad_pcb (KiCad board)
At the start: 2 copper layers, 150 x 200 mm, 45 parts, among them J0 Panel_GND_Solder_Wire_Pad

Commit message: Concluded core and resonance circuits design
Other:
- board text added: "1/1"
- board text added: "OFF"

Commit message: Changed Bus CV switch silkscreen
Parts:
- H12, H13, H17, H22, H28, H32: footprint SynthStuff:Pot_Cutout_Tiny_attv -> SynthStuff:Pot_Cutout_Tiny_attv_P110KH1
Other:
- board text removed: "Off"
- board text removed: "V/Oct"

Commit message: Updated switches symbols and fps
Parts:
- H14, H19, H20, H23, H24, H26, H33, H34, H35, H44: footprint SynthStuff:Toggle_Switch_Cutout -> SynthStuff:Toggle_Switch_TE_Cutout
