File: DMH_Dual_VCF_Diode_Ladder_PANEL/DMH_Dual_VCF_Diode_Ladder_PANEL.kicad_sch (KiCad schematic)
At the start: 20 parts, among them J0 Panel_GND_Solder_Wire_Pad

Commit message: Finished panel
Parts:
- removed H15: BP, SynthStuff:Toggle_Switch_Cutout, symbol SynthStuff:MountingHole_ToggleSwitch
- removed H16: HP, SynthStuff:Toggle_Switch_Cutout, symbol SynthStuff:MountingHole_ToggleSwitch
- added H15: CV 1, SynthStuff:Jack_6.35mm_Cutout_v3, symbol SynthStuff:MountingHole_Jack6.35mm_v2
- added H16: Input, SynthStuff:Jack_6.35mm_Cutout_v3, symbol SynthStuff:MountingHole_Jack6.35mm_v2
- added H20, H34: BP, SynthStuff:Toggle_Switch_Cutout, symbol SynthStuff:MountingHole_ToggleSwitch
- added H21: Drive, SynthStuff:Pot_Cutout_Small, symbol SynthStuff:MountingHole_Pot
- added H22: CV 1 Amt, SynthStuff:Pot_Cutout_Tiny, symbol SynthStuff:MountingHole_Pot
- added H23: Bus CV, SynthStuff:Toggle_Switch_Cutout, symbol SynthStuff:MountingHole_ToggleSwitch
- added H24: LP, SynthStuff:Toggle_Switch_Cutout, symbol SynthStuff:MountingHole_ToggleSwitch
- added H25: CV 2, SynthStuff:Jack_6.35mm_Cutout_v3, symbol SynthStuff:MountingHole_Jack6.35mm_v2
- added H26, H35: HP, SynthStuff:Toggle_Switch_Cutout, symbol SynthStuff:MountingHole_ToggleSwitch
- added H27: Cutoff, SynthStuff:Pot_Cutout_Large_v2, symbol SynthStuff:MountingHole_Pot
- added H28: (Bus) CV 2 Amt, SynthStuff:Pot_Cutout_Tiny, symbol SynthStuff:MountingHole_Pot
- added H29: CV 3, SynthStuff:Jack_6.35mm_Cutout_v3, symbol SynthStuff:MountingHole_Jack6.35mm_v2
- added H30: Output, SynthStuff:Jack_6.35mm_Cutout_Output_v6, symbol SynthStuff:MountingHole_Jack6.35mm_Output_v2
- added H31: Resonance, SynthStuff:Pot_Cutout_Small, symbol SynthStuff:MountingHole_Pot
- added H32: CV 3 Amt, SynthStuff:Pot_Cutout_Tiny, symbol SynthStuff:MountingHole_Pot
- added H33: Link, SynthStuff:Toggle_Switch_Cutout, symbol SynthStuff:MountingHole_ToggleSwitch
- added H36, H37, H38, H39: MountingHole_Rails, SynthStuff:MountingHole_Rails, symbol SynthStuff:MountingHole_Rails
- added H40: LED A, SynthStuff:MountingHole_LED_3mm, symbol Mechanical:MountingHole
- added H41: LED Link, SynthStuff:MountingHole_LED_3mm, symbol Mechanical:MountingHole
- added H42: LED B, SynthStuff:MountingHole_LED_3mm, symbol Mechanical:MountingHole
- H10, H11: footprint SynthStuff:Pot_Cutout_Medium -> SynthStuff:Pot_Cutout_Small
- H12: value CV 1 Amount -> CV 1 Amt
- H13: value CV 3 Amount -> CV 3 Amt
- H17: value (Bus) CV 2 Amount -> (Bus) CV 2 Amt
- H9: footprint SynthStuff:Pot_Cutout_Huge_v2 -> SynthStuff:Pot_Cutout_Large_v2
Connections:
- net GND: now also H15.1, H16.1, H20.1, H21.1, H22.1, H23.1, H24.1, H25.1, H26.1, H27.1, H28.1, H29.1, H30.1, H31.1, H32.1, H33.1, H34.1, H35.1, H36.1, H37.1, H38.1, H39.1
Other:
- moved on the sheet: H1, H10, H11, H12, H13, H14, H17, H18, H19, H2, H3, H4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

Commit message: Added central cutoff knob
Parts:
- added H43: Cutoff, SynthStuff:Pot_Cutout_Huge_v2, symbol SynthStuff:MountingHole_Pot
- H27, H9: footprint SynthStuff:Pot_Cutout_Large_v2 -> SynthStuff:Pot_Cutout_Small
Connections:
- net GND: now also H43.1
Changed lines of the file:
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@@
 	)
 	(junction
+		(at 25.4 114.3)
+		(diameter 0)
+		(color 0 0 0 0)
+	)
+	(junction
 		(at 27.94 241.3)
 		(diameter 0)
@@
 	(wire
 		(pts
+			(xy 101.6 54.61) (xy 101.6 63.5)
+		)
+		(stroke
+			(width 0)
+			(type default)
+		)
+	)
+	(wire
+		(pts
 			(xy 25.4 170.18) (xy 25.4 179.07)
 		)
@@
 	(wire
 		(pts
+			(xy 101.6 63.5) (xy 25.4 63.5)
+		)
+		(stroke
+			(width 0)
+			(type default)
+		)
+	)
+	(wire
+		(pts
 			(xy 25.4 114.3) (xy 25.4 139.7)
 		)
@@
 	(wire
 		(pts
+			(xy 25.4 63.5) (xy 25.4 114.3)
+		)
+		(stroke
+			(width 0)
+			(type default)
+		)
+	)
+	(wire
+		(pts
 			(xy 146.05 130.81) (xy 146.05 139.7)
 		)
@@
 	)
 	(symbol
+		(lib_id "SynthStuff:MountingHole_Pot")
+		(at 101.6 52.07 0)
+		(unit 1)
+		(exclude_from_sim yes)
+		(in_bom no)
+		(on_board yes)
+		(dnp no)
+		(fields_autoplaced yes)
+		(property "Reference" "H43"
+			(at 104.14 48.2599 0)
+			(effects
+				(font
+					(size 1.27 1.27)
+				)
+				(justify left)
+			)
+		)
+		(property "Value" "Cutoff"
+			(at 104.14 50.7999 0)
+			(effects
+				(font
+					(size 1.27 1.27)
+				)
+				(justify left)
+			)
+		)
+		(property "Footprint" "SynthStuff:Pot_Cutout_Huge_v2"
+			(at 101.6 52.07 0)
+			(effects
+				(font
+					(size 1.27 1.27)
+				)
+				(hide yes)
+			)
+		)
+		(property "Datasheet" "~"
+			(at 101.6 52.07 0)
+			(effects
+				(font
+					(size 1.27 1.27)
+				)
+				(hide yes)
+			)
+		)
+		(property "Description" "Pot Mounting Hole"
+			(at 104.14 53.3399 0)
+			(effects
+				(font
+					(size 1.27 1.27)
+				)
+				(justify left)
+			)
+		)
+		(property "Function" ""
+			(at 101.6 52.07 0)
+			(effects
+				(font
+					(size 1.27 1.27)
+				)
+			)
+		)
+		(pin "1"
+		)
+		(instances
+			(project "DMH_Dual_VCF_Diode_Ladder_PANEL"
+				(path "/a552705f-a9fe-462e-9913-5cfcc08b233c"
+					(reference "H43")
+					(unit 1)
+				)
+			)
+		)
+	)
+	(symbol
 		(lib_name "MountingHole_ToggleSwitch_1")
 		(lib_id "SynthStuff:MountingHole_ToggleSwitch")
@@
 			)
 		)
-		(property "Footprint" "SynthStuff:Pot_Cutout_Large_v2"
+		(property "Footprint" "SynthStuff:Pot_Cutout_Small"
 			(at 57.15 90.17 0)
 			(effects
@@
 			)
 		)
-		(property "Footprint" "SynthStuff:Pot_Cutout_Large_v2"
+		(property "Footprint" "SynthStuff:Pot_Cutout_Small"
 			(at 146.05 90.17 0)
 			(effects

Commit message: Changed features on panel
Parts:
- H13, H32: value CV 3 Amt -> Res CV Amt
- H17, H28: value (Bus) CV 2 Amt -> CV 2 Amt
- H27, H9: footprint SynthStuff:Pot_Cutout_Small -> SynthStuff:Pot_Cutout_Medium_v2
- H29, H7: value CV 3 -> Res CV
Changed lines of the file:
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@@
 			)
 		)
-		(property "Value" "CV 3"
+		(property "Value" "Res CV"
 			(at 72.39 203.1999 0)
 			(effects
@@
 			)
 		)
-		(property "Value" "CV 3 Amt"
+		(property "Value" "Res CV Amt"
 			(at 173.99 126.9999 0)
 			(effects
@@
 			)
 		)
-		(property "Footprint" "SynthStuff:Pot_Cutout_Small"
+		(property "Footprint" "SynthStuff:Pot_Cutout_Medium_v2"
 			(at 57.15 90.17 0)
 			(effects
@@
 			)
 		)
-		(property "Value" "CV 3 Amt"
+		(property "Value" "Res CV Amt"
 			(at 85.09 126.9999 0)
 			(effects
@@
 			)
 		)
-		(property "Value" "(Bus) CV 2 Amt"
+		(property "Value" "CV 2 Amt"
 			(at 59.69 126.9999 0)
 			(effects
@@
 			)
 		)
-		(property "Value" "(Bus) CV 2 Amt"
+		(property "Value" "CV 2 Amt"
 			(at 148.59 126.9999 0)
 			(effects
@@
 			)
 		)
-		(property "Value" "CV 3"
+		(property "Value" "Res CV"
 			(at 161.29 203.1999 0)
 			(effects
@@
 			)
 		)
-		(property "Footprint" "SynthStuff:Pot_Cutout_Small"
+		(property "Footprint" "SynthStuff:Pot_Cutout_Medium_v2"
 			(at 146.05 90.17 0)
 			(effects

Commit message: Reorganized panel
... and added Feed switch.
Parts:
- added H44: Feed, SynthStuff:Toggle_Switch_Cutout, symbol SynthStuff:MountingHole_ToggleSwitch
- H12, H13, H17, H22, H28, H32: footprint SynthStuff:Pot_Cutout_Tiny -> SynthStuff:Pot_Cutout_Tiny_attv
Connections:
- net GND: now also H44.1
Changed lines of the file:
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@@
 	)
 	(junction
+		(at 88.9 228.6)
+		(diameter 0)
+		(color 0 0 0 0)
+	)
+	(junction
 		(at 27.94 241.3)
 		(diameter 0)
@@
 	(wire
 		(pts
-			(xy 97.79 228.6) (xy 45.72 228.6)
+			(xy 97.79 228.6) (xy 88.9 228.6)
 		)
 		(stroke
@@
 	(wire
 		(pts
+			(xy 88.9 228.6) (xy 88.9 241.3)
+		)
+		(stroke
+			(width 0)
+			(type default)
+		)
+	)
+	(wire
+		(pts
 			(xy 24.13 251.46) (xy 27.94 251.46)
 		)
@@
 	(wire
 		(pts
+			(xy 88.9 228.6) (xy 45.72 228.6)
+		)
+		(stroke
+			(width 0)
+			(type default)
+		)
+	)
+	(wire
+		(pts
 			(xy 114.3 152.4) (xy 114.3 139.7)
 		)
@@
 	(wire
 		(pts
+			(xy 97.79 240.03) (xy 97.79 241.3)
+		)
+		(stroke
+			(width 0)
+			(type default)
+		)
+	)
+	(wire
+		(pts
 			(xy 146.05 130.81) (xy 146.05 139.7)
 		)
@@
 	(wire
 		(pts
+			(xy 97.79 241.3) (xy 88.9 241.3)
+		)
+		(stroke
+			(width 0)
+			(type default)
+		)
+	)
+	(wire
+		(pts
 			(xy 33.02 271.78) (xy 48.26 271.78)
 		)
@@
 			)
 		)
-		(property "Footprint" "SynthStuff:Pot_Cutout_Tiny"
+		(property "Footprint" "SynthStuff:Pot_Cutout_Tiny_attv"
 			(at 120.65 128.27 0)
 			(effects
@@
 			)
 		)
+		(property "Function" ""
+			(at 120.65 128.27 0)
+			(effects
+				(font
+					(size 1.27 1.27)
+				)
+			)
+		)
 		(pin "1"
 		)
@@
 			)
 		)
-		(property "Footprint" "SynthStuff:Pot_Cutout_Tiny"
+		(property "Footprint" "SynthStuff:Pot_Cutout_Tiny_attv"
 			(at 171.45 128.27 0)
 			(effects
@@
 			)
 		)
+		(property "Function" ""
+			(at 171.45 128.27 0)
+			(effects
+				(font
+					(size 1.27 1.27)
+				)
+			)
+		)
 		(pin "1"
 		)
@@
 			)
 		)
-		(property "Footprint" "SynthStuff:Pot_Cutout_Tiny"
+		(property "Footprint" "SynthStuff:Pot_Cutout_Tiny_attv"
 			(at 31.75 128.27 0)
 			(effects
@@
 			)
 		)
+		(property "Function" ""
+			(at 31.75 128.27 0)
+			(effects
+				(font
+					(size 1.27 1.27)
+				)
+			)
+		)
 		(pin "1"
 		)
@@
 			)
 		)
-		(property "Footprint" "SynthStuff:Pot_Cutout_Tiny"
+		(property "Footprint" "SynthStuff:Pot_Cutout_Tiny_attv"
 			(at 82.55 128.27 0)
 			(effects
@@
 			)
 		)
+		(property "Function" ""
+			(at 82.55 128.27 0)
+			(effects
+				(font
+					(size 1.27 1.27)
+				)
+			)
+		)
 		(pin "1"
 		)
@@
 	)
 	(symbol
+		(lib_name "MountingHole_ToggleSwitch_1")
+		(lib_id "SynthStuff:MountingHole_ToggleSwitch")
+		(at 97.79 236.22 0)
+		(unit 1)
+		(exclude_from_sim yes)
+		(in_bom no)
+		(on_board yes)
+		(dnp no)
+		(property "Reference" "H44"
+			(at 100.33 234.9499 0)
+			(effects
+				(font
+					(size 1.27 1.27)
+				)
+				(justify left)
+			)
+		)
+		(property "Value" "Feed"
+			(at 100.33 237.4899 0)
+			(effects
+				(font
+					(size 1.27 1.27)
+				)
+				(justify left)
+			)
+		)
+		(property "Footprint" "SynthStuff:Toggle_Switch_Cutout"
+			(at 97.79 236.22 0)
+			(effects
+				(font
+					(size 1.27 1.27)
+				)
+				(hide yes)
+			)
+		)
+		(property "Datasheet" "~"
+			(at 97.79 236.22 0)
+			(effects
+				(font
+					(size 1.27 1.27)
+				)
+				(hide yes)
+			)
+		)
+		(property "Description" "Toggle Switch Mounting Hole"
+			(at 100.584 240.03 0)
+			(effects
+				(font
+					(size 1.27 1.27)
+				)
+				(justify left)
+			)
+		)
+		(property "Function" "Bus CV"
+			(at 101.6 239.776 0)
+			(effects
+				(font
+					(size 1.27 1.27)
+					(thickness 0.1588)
+				)
+				(hide yes)
+			)
+		)
+		(pin "1"
+		)
+		(instances
+			(project "DMH_Dual_VCF_Diode_Ladder_PANEL"
+				(path "/a552705f-a9fe-462e-9913-5cfcc08b233c"
+					(reference "H44")
+					(unit 1)
+				)
+			)
+		)
+	)
+	(symbol
 		(lib_id "SynthStuff:MountingHole_Rails")
 		(at 27.94 247.65 0)
@@
 			)
 		)
-		(property "Footprint" "SynthStuff:Pot_Cutout_Tiny"
+		(property "Footprint" "SynthStuff:Pot_Cutout_Tiny_attv"
 			(at 57.15 128.27 0)
 			(effects
@@
 			)
 		)
+		(property "Function" ""
+			(at 57.15 128.27 0)
+			(effects
+				(font
+					(size 1.27 1.27)
+				)
+			)
+		)
 		(pin "1"
 		)
@@
 			)
 		)
-		(property "Footprint" "SynthStuff:Pot_Cutout_Tiny"
+		(property "Footprint" "SynthStuff:Pot_Cutout_Tiny_attv"
 			(at 146.05 128.27 0)
 			(effects
@@
 			)
 		)
+		(property "Function" ""
+			(at 146.05 128.27 0)
+			(effects
+				(font
+					(size 1.27 1.27)
+				)
+			)
+		)

Commit message: Generated BoM
Parts:
- H10, H11, H12, H13, H17, H21, H22, H27, H28, H31, H32, H43, H9: now in the parts list
Changed lines of the file:
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@@
 	)
 	(symbol
-		(lib_name "MountingHole_ToggleSwitch_1")
 		(lib_id "SynthStuff:MountingHole_ToggleSwitch")
 		(at 120.65 148.59 0)
@@
 		(unit 1)
 		(exclude_from_sim yes)
-		(in_bom no)
+		(in_bom yes)
 		(on_board yes)
 		(dnp no)
@@
 		(unit 1)
 		(exclude_from_sim yes)
-		(in_bom no)
+		(in_bom yes)
 		(on_board yes)
 		(dnp no)
@@
 		(unit 1)
 		(exclude_from_sim yes)
-		(in_bom no)
+		(in_bom yes)
 		(on_board yes)
 		(dnp no)
@@
 		(unit 1)
 		(exclude_from_sim yes)
-		(in_bom no)
+		(in_bom yes)
 		(on_board yes)
 		(dnp no)
@@
 	)
 	(symbol
-		(lib_name "MountingHole_ToggleSwitch_1")
 		(lib_id "SynthStuff:MountingHole_ToggleSwitch")
 		(at 31.75 175.26 0)
@@
 		(unit 1)
 		(exclude_from_sim yes)
-		(in_bom no)
+		(in_bom yes)
 		(on_board yes)
 		(dnp no)
@@
 	)
 	(symbol
-		(lib_name "MountingHole_ToggleSwitch_1")
 		(lib_id "SynthStuff:MountingHole_ToggleSwitch")
 		(at 31.75 148.59 0)
@@
 	)
 	(symbol
-		(lib_name "MountingHole_ToggleSwitch_1")
 		(lib_id "SynthStuff:MountingHole_ToggleSwitch")
 		(at 97.79 223.52 0)
@@
 		(unit 1)
 		(exclude_from_sim yes)
-		(in_bom no)
+		(in_bom yes)
 		(on_board yes)
 		(dnp no)
@@
 		(unit 1)
 		(exclude_from_sim yes)
-		(in_bom no)
+		(in_bom yes)
 		(on_board yes)
 		(dnp no)
@@
 		(unit 1)
 		(exclude_from_sim yes)
-		(in_bom no)
+		(in_bom yes)
 		(on_board yes)
 		(dnp no)
@@
 	)
 	(symbol
-		(lib_name "MountingHole_ToggleSwitch_1")
 		(lib_id "SynthStuff:MountingHole_ToggleSwitch")
 		(at 31.75 157.48 0)
@@
 	)
 	(symbol
-		(lib_name "MountingHole_ToggleSwitch_1")
 		(lib_id "SynthStuff:MountingHole_ToggleSwitch")
 		(at 120.65 166.37 0)
@@
 	)
 	(symbol
-		(lib_name "MountingHole_ToggleSwitch_1")
 		(lib_id "SynthStuff:MountingHole_ToggleSwitch")
 		(at 97.79 236.22 0)
@@
 		(unit 1)
 		(exclude_from_sim yes)
-		(in_bom no)
+		(in_bom yes)
 		(on_board yes)
 		(dnp no)
@@
 	)
 	(symbol
-		(lib_name "MountingHole_ToggleSwitch_1")
 		(lib_id "SynthStuff:MountingHole_ToggleSwitch")
 		(at 120.65 157.48 0)
@@
 		(unit 1)
 		(exclude_from_sim yes)
-		(in_bom no)
+		(in_bom yes)
 		(on_board yes)
 		(dnp no)
@@
 	)
 	(symbol
-		(lib_name "MountingHole_ToggleSwitch_1")
 		(lib_id "SynthStuff:MountingHole_ToggleSwitch")
 		(at 31.75 166.37 0)
@@
 		(unit 1)
 		(exclude_from_sim yes)
-		(in_bom no)
+		(in_bom yes)
 		(on_board yes)
 		(dnp no)
@@
 		(unit 1)
 		(exclude_from_sim yes)
-		(in_bom no)
+		(in_bom yes)
 		(on_board yes)
 		(dnp no)
@@
 		(unit 1)
 		(exclude_from_sim yes)
-		(in_bom no)
+		(in_bom yes)
 		(on_board yes)
 		(dnp no)
@@
 	)
 	(symbol
-		(lib_name "MountingHole_ToggleSwitch_1")
 		(lib_id "SynthStuff:MountingHole_ToggleSwitch")
 		(at 120.65 175.26 0)

Commit message: Changed Bus CV switch silkscreen
Parts:
- H12, H13, H17, H22, H28, H32: footprint SynthStuff:Pot_Cutout_Tiny_attv -> SynthStuff:Pot_Cutout_Tiny_attv_P110KH1
Changed lines of the file:
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@@
 			)
 		)
-		(property "Footprint" "SynthStuff:Pot_Cutout_Tiny_attv"
+		(property "Footprint" "SynthStuff:Pot_Cutout_Tiny_attv_P110KH1"
 			(at 120.65 128.27 0)
 			(effects
@@
 			)
 		)
-		(property "Footprint" "SynthStuff:Pot_Cutout_Tiny_attv"
+		(property "Footprint" "SynthStuff:Pot_Cutout_Tiny_attv_P110KH1"
 			(at 171.45 128.27 0)
 			(effects
@@
 			)
 		)
-		(property "Footprint" "SynthStuff:Pot_Cutout_Tiny_attv"
+		(property "Footprint" "SynthStuff:Pot_Cutout_Tiny_attv_P110KH1"
 			(at 31.75 128.27 0)
 			(effects
@@
 			)
 		)
-		(property "Footprint" "SynthStuff:Pot_Cutout_Tiny_attv"
+		(property "Footprint" "SynthStuff:Pot_Cutout_Tiny_attv_P110KH1"
 			(at 82.55 128.27 0)
 			(effects
@@
 			)
 		)
-		(property "Footprint" "SynthStuff:Pot_Cutout_Tiny_attv"
+		(property "Footprint" "SynthStuff:Pot_Cutout_Tiny_attv_P110KH1"
 			(at 57.15 128.27 0)
 			(effects
@@
 			)
 		)
-		(property "Footprint" "SynthStuff:Pot_Cutout_Tiny_attv"
+		(property "Footprint" "SynthStuff:Pot_Cutout_Tiny_attv_P110KH1"
 			(at 146.05 128.27 0)
 			(effects

Commit message: Updated switches symbols and fps
Parts:
- H14, H19, H20, H23, H24, H26, H33, H34, H35, H44: footprint SynthStuff:Toggle_Switch_Cutout -> SynthStuff:Toggle_Switch_TE_Cutout
Changed lines of the file:
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@@
 			)
 		)
-		(property "Footprint" "SynthStuff:Toggle_Switch_Cutout"
+		(property "Footprint" "SynthStuff:Toggle_Switch_TE_Cutout"
 			(at 120.65 148.59 0)
 			(effects
@@
 			)
 		)
-		(property "Footprint" "SynthStuff:Toggle_Switch_Cutout"
+		(property "Footprint" "SynthStuff:Toggle_Switch_TE_Cutout"
 			(at 31.75 175.26 0)
 			(effects
@@
 			)
 		)
-		(property "Footprint" "SynthStuff:Toggle_Switch_Cutout"
+		(property "Footprint" "SynthStuff:Toggle_Switch_TE_Cutout"
 			(at 31.75 148.59 0)
 			(effects
@@
 			)
 		)
-		(property "Footprint" "SynthStuff:Toggle_Switch_Cutout"
+		(property "Footprint" "SynthStuff:Toggle_Switch_TE_Cutout"
 			(at 97.79 223.52 0)
 			(effects
@@
 			)
 		)
-		(property "Footprint" "SynthStuff:Toggle_Switch_Cutout"
+		(property "Footprint" "SynthStuff:Toggle_Switch_TE_Cutout"
 			(at 31.75 157.48 0)
 			(effects
@@
 			)
 		)
-		(property "Footprint" "SynthStuff:Toggle_Switch_Cutout"
+		(property "Footprint" "SynthStuff:Toggle_Switch_TE_Cutout"
 			(at 120.65 166.37 0)
 			(effects
@@
 			)
 		)
-		(property "Footprint" "SynthStuff:Toggle_Switch_Cutout"
+		(property "Footprint" "SynthStuff:Toggle_Switch_TE_Cutout"
 			(at 97.79 236.22 0)
 			(effects
@@
 			)
 		)
-		(property "Footprint" "SynthStuff:Toggle_Switch_Cutout"
+		(property "Footprint" "SynthStuff:Toggle_Switch_TE_Cutout"
 			(at 120.65 157.48 0)
 			(effects
@@
 			)
 		)
-		(property "Footprint" "SynthStuff:Toggle_Switch_Cutout"
+		(property "Footprint" "SynthStuff:Toggle_Switch_TE_Cutout"
 			(at 31.75 166.37 0)
 			(effects
@@
 			)
 		)
-		(property "Footprint" "SynthStuff:Toggle_Switch_Cutout"
+		(property "Footprint" "SynthStuff:Toggle_Switch_TE_Cutout"
 			(at 120.65 175.26 0)
 			(effects
